File: pcb/hackpad.kicad_pcb (KiCad board)
At the start: 2 copper layers, 46.5 x 59 mm, 6 parts, among them SW1 SW_Push, SW2 SW_Push, SW3 SW_Push, SW4 SW_Push, SW5 RotaryEncoder, U1 MOUDLE-SEEEDUINO-XIAO

Commit message: Added rotary encoder to cad folder, added gap for usb port
Parts:
- moved U1 0.19 mm to (140.0, 76.7)
Routing:
- net Net-(U1-PA9_A5_D5_SCL): track 74.3 -> 98.2 mm
Other:
- board size 46.5 x 59 mm -> 43.5 x 59 mm
Changed lines of the file:
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@@
 	(footprint "RF_Module:MCU_Seeed_ESP32C3"
 		(layer "B.Cu")
-		(at 140.1 76.6 90)
+		(at 139.96 76.73 90)
 		(descr "ESP32C3 Seeed Xiao RF Wifi Shield (https://www.seeedstudio.com/blog/wp-content/uploads/2022/08/Seeed-Studio-XIAO-Series-Package-and-PCB-Design.pdf)")
 		(tags "wifi bluetooth microcontroller")
 		(property "Reference" "U1"
-			(at 7 12 270)
+			(at 12.6 6.9 270)
 			(unlocked yes)
 			(layer "B.SilkS")
@@
 	(gr_rect
 		(start 107 49.5)
-		(end 153.5 108.5)
+		(end 150.5 108.5)
 		(stroke
 			(width 0.05)
@@
 	)
 	(segment
-		(start 150 89.13137)
-		(end 144.76637 94.365)
+		(start 134.88 85.23)
+		(end 134.88 89.685685)
 		(width 0.2)
 		(layer "B.Cu")
@@
 	)
 	(segment
-		(start 138.540101 94.365)
-		(end 135.02 90.844899)
+		(start 113.334314 101.9)
+		(end 110.6 99.165685)
 		(width 0.2)
 		(layer "B.Cu")
@@
 	)
 	(segment
-		(start 128.525 55.375)
-		(end 140.940685 55.375)
+		(start 122.665685 101.9)
+		(end 113.334314 101.9)
 		(width 0.2)
 		(layer "B.Cu")
@@
 	)
 	(segment
-		(start 150 64.434315)
-		(end 150 89.13137)
+		(start 110.6 55.9)
+		(end 113.335 53.165)
 		(width 0.2)
 		(layer "B.Cu")
@@
 	)
 	(segment
-		(start 140.940685 55.375)
-		(end 150 64.434315)
+		(start 113.335 53.165)
+		(end 126.315 53.165)
 		(width 0.2)
 		(layer "B.Cu")
@@
 	)
 	(segment
-		(start 135.02 90.844899)
-		(end 135.02 85.1)
+		(start 134.88 89.685685)
+		(end 122.665685 101.9)
 		(width 0.2)
 		(layer "B.Cu")
@@
 	)
 	(segment
-		(start 144.76637 94.365)
-		(end 138.540101 94.365)
+		(start 126.315 53.165)
+		(end 128.525 55.375)
+		(width 0.2)
+		(layer "B.Cu")
+		(net "Net-(U1-PA9_A5_D5_SCL)")
+	)
+	(segment
+		(start 110.6 99.165685)
+		(end 110.6 55.9)
 		(width 0.2)
 		(layer "B.Cu")
@@
 		(polygon
 			(pts
-				(xy 107 49.5) (xy 107 108.5) (xy 153.5 108.5) (xy 153.5 49.5)
-			)
-		)
+				(xy 107 49.5) (xy 107 108.5) (xy 150.5 108.5) (xy 150.5 81) (xy 149.5 81) (xy 149.5 72.5) (xy 150.5 72.5)
+				(xy 150.5 49.5)
+			)
+		)
